File: Hardware/5x3 Minibadge front board/minibadge_grid.kicad_sch (KiCad schematic)
At the start: 15 parts

Commit message: small chages
Parts:
- renumbered MB14 to MB10, MB3 to MB11, MB6 to MB12, MB9 to MB13, MB12 to MB14, MB4 to MB2, MB7 to MB3, MB10 to MB4, MB13 to MB5, MB2 to MB6, MB5 to MB7, MB11 to MB9
Changed lines of the file:
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@@
 		(on_board yes)
 		(dnp no)
-		(property "Reference" "MB9"
+		(property "Reference" "MB13"
 			(at 96.774 137.16 0)
 			(effects
@@
 			(project "Minibadge Display 5x3"
 				(path "/e5119d15-74fb-4259-abbc-5cab1f368532/6e97fb62-2d35-4554-a843-3cbb1f9f2f26"
-					(reference "MB9")
+					(reference "MB13")
 					(unit 1)
 				)
@@
 		(on_board yes)
 		(dnp no)
-		(property "Reference" "MB4"
+		(property "Reference" "MB2"
 			(at 68.834 53.34 0)
 			(effects
@@
 			(project "Minibadge Display 5x3"
 				(path "/e5119d15-74fb-4259-abbc-5cab1f368532/6e97fb62-2d35-4554-a843-3cbb1f9f2f26"
-					(reference "MB4")
+					(reference "MB2")
 					(unit 1)
 				)
@@
 		(on_board yes)
 		(dnp no)
-		(property "Reference" "MB13"
+		(property "Reference" "MB5"
 			(at 152.654 53.34 0)
 			(effects
@@
 			(project "Minibadge Display 5x3"
 				(path "/e5119d15-74fb-4259-abbc-5cab1f368532/6e97fb62-2d35-4554-a843-3cbb1f9f2f26"
-					(reference "MB13")
+					(reference "MB5")
 					(unit 1)
 				)
@@
 		(on_board yes)
 		(dnp no)
-		(property "Reference" "MB6"
+		(property "Reference" "MB12"
 			(at 68.834 137.16 0)
 			(effects
@@
 			(project "Minibadge Display 5x3"
 				(path "/e5119d15-74fb-4259-abbc-5cab1f368532/6e97fb62-2d35-4554-a843-3cbb1f9f2f26"
-					(reference "MB6")
+					(reference "MB12")
 					(unit 1)
 				)
@@
 		(on_board yes)
 		(dnp no)
-		(property "Reference" "MB10"
+		(property "Reference" "MB4"
 			(at 124.714 53.34 0)
 			(effects
@@
 			(project "Minibadge Display 5x3"
 				(path "/e5119d15-74fb-4259-abbc-5cab1f368532/6e97fb62-2d35-4554-a843-3cbb1f9f2f26"
-					(reference "MB10")
+					(reference "MB4")
 					(unit 1)
 				)
@@
 		(on_board yes)
 		(dnp no)
-		(property "Reference" "MB12"
+		(property "Reference" "MB14"
 			(at 124.714 137.16 0)
 			(effects
@@
 			(project "Minibadge Display 5x3"
 				(path "/e5119d15-74fb-4259-abbc-5cab1f368532/6e97fb62-2d35-4554-a843-3cbb1f9f2f26"
-					(reference "MB12")
+					(reference "MB14")
 					(unit 1)
 				)
@@
 		(on_board yes)
 		(dnp no)
-		(property "Reference" "MB7"
+		(property "Reference" "MB3"
 			(at 96.774 53.34 0)
 			(effects
@@
 			(project "Minibadge Display 5x3"
 				(path "/e5119d15-74fb-4259-abbc-5cab1f368532/6e97fb62-2d35-4554-a843-3cbb1f9f2f26"
-					(reference "MB7")
+					(reference "MB3")
 					(unit 1)
 				)
@@
 		(on_board yes)
 		(dnp no)
-		(property "Reference" "MB14"
+		(property "Reference" "MB10"
 			(at 152.654 95.25 0)
 			(effects
@@
 			(project "Minibadge Display 5x3"
 				(path "/e5119d15-74fb-4259-abbc-5cab1f368532/6e97fb62-2d35-4554-a843-3cbb1f9f2f26"
-					(reference "MB14")
+					(reference "MB10")
 					(unit 1)
 				)
@@
 		(on_board yes)
 		(dnp no)
-		(property "Reference" "MB2"
+		(property "Reference" "MB6"
 			(at 40.894 95.25 0)
 			(effects
@@
 			(project "Minibadge Display 5x3"
 				(path "/e5119d15-74fb-4259-abbc-5cab1f368532/6e97fb62-2d35-4554-a843-3cbb1f9f2f26"
-					(reference "MB2")
+					(reference "MB6")
 					(unit 1)
 				)
@@
 		(on_board yes)
 		(dnp no)
-		(property "Reference" "MB3"
+		(property "Reference" "MB11"
 			(at 40.894 137.16 0)
 			(effects
@@
 			(project "Minibadge Display 5x3"
 				(path "/e5119d15-74fb-4259-abbc-5cab1f368532/6e97fb62-2d35-4554-a843-3cbb1f9f2f26"
-					(reference "MB3")
+					(reference "MB11")
 					(unit 1)
 				)
@@
 		(on_board yes)
 		(dnp no)
-		(property "Reference" "MB11"
+		(property "Reference" "MB9"
 			(at 124.714 95.25 0)
 			(effects
@@
 			(project "Minibadge Display 5x3"
 				(path "/e5119d15-74fb-4259-abbc-5cab1f368532/6e97fb62-2d35-4554-a843-3cbb1f9f2f26"
-					(reference "MB11")
+					(reference "MB9")
 					(unit 1)
 				)
@@
 		(on_board yes)
 		(dnp no)
-		(property "Reference" "MB5"
+		(property "Reference" "MB7"
 			(at 68.834 95.25 0)
 			(effects
@@
 			(project "Minibadge Display 5x3"
 				(path "/e5119d15-74fb-4259-abbc-5cab1f368532/6e97fb62-2d35-4554-a843-3cbb1f9f2f26"
-					(reference "MB5")
+					(reference "MB7")
 					(unit 1)
 				)
