File: Hardware/Main board/RP2040.kicad_sch (KiCad schematic)
At the start: 19 parts, among them U2 ABM8-272-T3, U4 RP2040

Commit message: Finish routing
Connections:
- net +1V1: no longer U4.23 (DVDD), U4.45 (VREG_VOUT), U4.50 (DVDD)
- new net: U4.23 (DVDD), U4.50 (DVDD)
Changed lines of the file:
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@@
 	)
 	(junction
-		(at 101.6 58.42)
-		(diameter 0)
-		(color 0 0 0 0)
-	)
-	(junction
 		(at 134.62 41.91)
 		(diameter 0)
@@
 	)
 	(junction
-		(at 101.6 62.23)
-		(diameter 0)
-		(color 0 0 0 0)
-	)
-	(junction
 		(at 204.47 41.91)
 		(diameter 0)
@@
 	(wire
 		(pts
-			(xy 104.14 64.77) (xy 104.14 62.23)
-		)
-		(stroke
-			(width 0)
-			(type default)
-		)
-	)
-	(wire
-		(pts
 			(xy 132.08 92.71) (xy 154.94 92.71)
 		)
@@
 	(wire
 		(pts
-			(xy 104.14 62.23) (xy 101.6 62.23)
-		)
-		(stroke
-			(width 0)
-			(type default)
-		)
-	)
-	(wire
-		(pts
 			(xy 77.47 95.25) (xy 81.28 95.25)
 		)
@@
 	(wire
 		(pts
-			(xy 101.6 62.23) (xy 101.6 64.77)
-		)
-		(stroke
-			(width 0)
-			(type default)
-		)
-	)
-	(wire
-		(pts
 			(xy 116.84 41.91) (xy 116.84 58.42)
 		)
@@
 	(wire
 		(pts
-			(xy 101.6 58.42) (xy 101.6 62.23)
-		)
-		(stroke
-			(width 0)
-			(type default)
-		)
-	)
-	(wire
-		(pts
 			(xy 132.08 85.09) (xy 154.94 85.09)
 		)
@@
 		(exclude_from_sim no)
 		(in_bom yes)
-		(on_board yes)
+		(on_board no)
 		(dnp no)
 		(property "Reference" "C10"
@@
 		(exclude_from_sim no)
 		(in_bom yes)
-		(on_board yes)
+		(on_board no)
 		(dnp no)
 		(fields_autoplaced yes)
@@
 		(exclude_from_sim no)
 		(in_bom yes)
-		(on_board yes)
+		(on_board no)
 		(dnp no)
 		(fields_autoplaced yes)
@@
 		(exclude_from_sim no)
 		(in_bom yes)
-		(on_board yes)
+		(on_board no)
 		(dnp no)
 		(property "Reference" "C9"
@@
 		(exclude_from_sim no)
 		(in_bom yes)
-		(on_board yes)
+		(on_board no)
 		(dnp no)
 		(fields_autoplaced yes)
@@
 		(exclude_from_sim no)
 		(in_bom yes)
-		(on_board yes)
+		(on_board no)
 		(dnp no)
 		(fields_autoplaced yes)
