File: Hardware/Main board/Flash.kicad_sch (KiCad schematic)
At the start: 4 parts, among them U10 W25Q32JVSS

Commit message: refactor PCB for new BMS layout
Parts:
- JP2: renamed from JP3; value USB_BOOT -> USB BOOT
- renumbered C7 to C10, R5 to R6, U10 to U2
Connections:
- net GND renamed AGND

Commit message: Add button and LEDs
Parts:
- removed JP2: USB BOOT, Jumper:SolderJumper-2_P1.3mm_Open_RoundedPad1.0x1.5mm, symbol Jumper:Jumper_2_Open
- added SW1: USB BOOT, Button_Switch_SMD:SW_Push_1P1T_XKB_TS-1187A, symbol Switch:SW_Push
Connections:
- net AGND: now also SW1.2
- net USB_BOOT: now also SW1.1
Changed lines of the file:
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@@
 	)
 	(symbol
-		(lib_id "Jumper:Jumper_2_Open")
+		(lib_id "Switch:SW_Push")
 		(at 116.84 81.28 270)
-		(mirror x)
 		(unit 1)
-		(exclude_from_sim yes)
-		(in_bom no)
+		(exclude_from_sim no)
+		(in_bom yes)
 		(on_board yes)
 		(dnp no)
 		(fields_autoplaced yes)
-		(property "Reference" "JP2"
-			(at 111.76 81.28 0)
+		(property "Reference" "SW1"
+			(at 120.65 80.0099 90)
 			(effects
 				(font
 					(size 1.27 1.27)
 				)
+				(justify left)
 			)
 		)
 		(property "Value" "USB BOOT"
-			(at 114.3 81.28 0)
+			(at 120.65 82.5499 90)
 			(effects
 				(font
 					(size 1.27 1.27)
 				)
+				(justify left)
 			)
 		)
-		(property "Footprint" "Jumper:SolderJumper-2_P1.3mm_Open_RoundedPad1.0x1.5mm"
-			(at 116.84 81.28 0)
+		(property "Footprint" "Button_Switch_SMD:SW_Push_1P1T_XKB_TS-1187A"
+			(at 121.92 81.28 0)
 			(effects
 				(font
@@
 		)
 		(property "Datasheet" "~"
-			(at 116.84 81.28 0)
+			(at 121.92 81.28 0)
 			(effects
 				(font
@@
 			)
 		)
-		(property "Description" "Jumper, 2-pole, open"
-			(at 116.84 81.28 0)
-			(effects
-				(font
-					(size 1.27 1.27)
-				)
-				(hide yes)
-			)
-		)
-		(property "Design guide" ""
+		(property "Description" "Push button switch, generic, two pins"
 			(at 116.84 81.28 0)
 			(effects
@@
 			(project ""
 				(path "/e5119d15-74fb-4259-abbc-5cab1f368532/72dbc5c2-e6c3-4b41-8ecd-db82b0a9ba3e"
-					(reference "JP2")
+					(reference "SW1")
 					(unit 1)
 				)

Commit message: swap diode footprint + add new part numbers
Parts:
- SW1: LCSC Part # (none) -> C318884
Changed lines of the file:
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@@
+			)
+		)
+		(property "JLCPCB Parts URL" ""
+			(at 116.84 81.28 0)
+			(effects
+				(font
+					(size 1.27 1.27)
+				)
+				(hide yes)
+			)
+		)
+		(property "LCSC Part #" "C318884"
+			(at 116.84 81.28 0)
+			(effects
+				(font
+					(size 1.27 1.27)
+				)
+				(hide yes)
+			)
+		)
+		(property "Design guide" ""
+			(at 116.84 81.28 0)
+			(effects
+				(font
+					(size 1.27 1.27)
+				)
+				(hide yes)
 			)
 		)
