File: Hardware/Main board/USB Switch.kicad_sch (KiCad schematic)
At the start: 2 parts

Commit message: Big changes
- Folder changes
- change dimensions of board to match thicker material
- begin part selection/footprint selection
Parts:
- C8: footprint (none) -> Capacitor_SMD:C_0402_1005Metric
Changed lines of the file:
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@@
 			)
 		)
-		(property "Footprint" ""
+		(property "Footprint" "Capacitor_SMD:C_0402_1005Metric"
 			(at 162.56 72.39 0)
 			(effects

Commit message: Part selection
Parts:
- U3: value ~ -> TS3USB221A; JLCPCB Part # (none) -> C128396; LCSC Part # (none) -> C128396
Changed lines of the file:
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@@
 			)
 		)
-		(property "Value" "~"
+		(property "Value" "TS3USB221A"
 			(at 146.9741 78.74 0)
 			(effects
@@
 			(at 144.78 81.28 0)
 			(effects
+				(font
+					(size 1.27 1.27)
+				)
+				(hide yes)
+			)
+		)
+		(property "JLCPCB Part #" "C128396"
+			(at 144.78 81.28 0)
+			(effects
+				(font
+					(size 1.27 1.27)
+				)
+				(hide yes)
+			)
+		)
+		(property "LCSC Part #" "C128396"
+			(at 144.78 81.28 0)
+			(effects

Commit message: refactor PCB for new BMS layout
Parts:
- renumbered C8 to C11
Connections:
- net GND renamed PGND
