File: Hardware/Main board/BMS.kicad_sch (KiCad schematic)
At the start: 24 parts, among them J2 BATT JST, U1 BQ25895

Commit message: Exclude BMS Reset from BOM
Parts:
- JP1: now left out of the parts list
Changed lines of the file:
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@@
 		(unit 1)
 		(exclude_from_sim yes)
-		(in_bom yes)
+		(in_bom no)
 		(on_board yes)
 		(dnp no)
